File: Schem/MorningJoe/pBITzBusInterface.kicad_sch (KiCad schematic)
At the start: 1 part, among them J5 pBITzBus

Commit message: Added both the Morning Joe and the Lunch Crema schematics, PCB, and KiCad library files.
Changed lines of the file:
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@@
+	)
+	(junction
+		(at 146.05 171.45)
+		(diameter 0)
+		(color 0 0 0 0)
 	)
 	(junction
@@
 	)
 	(junction
-		(at 228.6 133.35)
-		(diameter 0)
-		(color 0 0 0 0)
-	)
-	(junction
 		(at 228.6 142.24)
 		(diameter 0)
@@
 	(wire
 		(pts
+			(xy 146.05 171.45) (xy 149.86 171.45)
+		)
+		(stroke
+			(width 0)
+			(type default)
+		)
+	)
+	(wire
+		(pts
 			(xy 234.95 144.78) (xy 228.6 144.78)
 		)
@@
 	(wire
 		(pts
-			(xy 228.6 128.27) (xy 228.6 133.35)
+			(xy 228.6 128.27) (xy 228.6 142.24)
 		)
 		(stroke
@@
 		(pts
 			(xy 274.32 128.27) (xy 274.32 142.24)
-		)
-		(stroke
-			(width 0)
-			(type default)
-		)
-	)
-	(wire
-		(pts
-			(xy 228.6 133.35) (xy 228.6 142.24)
 		)
 		(stroke
@@
 		(shape output)
 		(at 146.05 194.31 0)
+		(effects
+			(font
+				(size 1.27 1.27)
+			)
+			(justify left)
+		)
+	)
+	(hierarchical_label "D0"
+		(shape bidirectional)
+		(at 149.86 171.45 0)
 		(effects
 			(font
@@
 					(unit 1)
 				)
-			)
-		)
-	)
-	(symbol
-		(lib_id "power:PWR_FLAG")
-		(at 228.6 133.35 90)
-		(unit 1)
-		(body_style 1)
-		(exclude_from_sim no)
-		(in_bom yes)
-		(on_board yes)
-		(in_pos_files yes)
-		(dnp no)
-		(fields_autoplaced yes)
-		(property "Reference" "#FLG01"
-			(at 226.695 133.35 0)
-			(hide yes)
-			(show_name no)
-			(do_not_autoplace no)
-			(effects
-				(font
-					(size 1.27 1.27)
-				)
-			)
-		)
-		(property "Value" "PWR_FLAG"
-			(at 224.79 133.3499 90)
-			(show_name no)
-			(do_not_autoplace no)
-			(effects
-				(font
-					(size 1.27 1.27)
-				)
-				(justify left)
-			)
-		)
-		(property "Footprint" ""
-			(at 228.6 133.35 0)
-			(hide yes)
-			(show_name no)
-			(do_not_autoplace no)
-			(effects
-				(font
-					(size 1.27 1.27)
-				)
-			)
-		)
-		(property "Datasheet" ""
-			(at 228.6 133.35 0)
-			(hide yes)
-			(show_name no)
-			(do_not_autoplace no)
-			(effects
-				(font
-					(size 1.27 1.27)
-				)
-			)
-		)
-		(property "Description" "Special symbol for telling ERC where power comes from"
-			(at 228.6 133.35 0)
-			(hide yes)
-			(show_name no)
-			(do_not_autoplace no)
-			(effects
-				(font
-					(size 1.27 1.27)
-				)
-			)
-		)
-		(pin "1"
-		)
-		(instances
-			(project "Zephyr-80-IO"
-				(path "/db33a8e4-587d-4e74-8d3f-b68910957121/61c97d6f-c0cd-4540-8832-42e8c844ef6d"
-					(reference "#FLG01")
-					(unit 1)
-				)
-			)
-			(project "MorningJoe"
-				(path "/e7f44da3-512d-42ef-9079-a376a3e5a592/84cc0ab2-d0b3-4bd4-8111-af5aef572a2e"
-					(reference "#FLG01")
-					(unit 1)
-				)
