File: Schem/MorningJoe/Video.kicad_sch (KiCad schematic)
At the start: 41 parts, among them J1 DE15_Socket_HighDensity_Mount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, U1 CD74HC139M96, U10 AS7C256A-10TCN, U2 TMS9928A, U3 SN74HC273DWR, U4 SN74HCT04DR, U5 SN74LVC1G19DCKR, U6 THS7314DR, U7 SN74HCT574DWR, U8 SN74HCT574DWR, U9 SN74HCT574DWR, Y1 MP107-E

Commit message: Added both the Morning Joe and the Lunch Crema schematics, PCB, and KiCad library files.
Parts:
- removed D1, D2: BAT54JW-7-F, Diode_SMD:D_SOD-323F, symbol Diode:BAT54J
- removed R1: 4K7, Resistor_SMD:R_0603_1608Metric, symbol Device:R
- removed U10: AS7C256A-10TCN, Footprints:TSOP-28_8X13P4_ALL, symbol 2026-01-18_07-40-02:AS7C256A-10TCN
- removed U4: SN74HCT04DR, Package_SO:SOIC-14_3.9x8.7mm_P1.27mm, symbol 74xx:74HC04
- removed U7, U8, U9: SN74HCT574DWR, Package_SO:SOIC-20W_7.5x12.8mm_P1.27mm, symbol 74xx:74LS574
- added C23: 220u, Capacitor_THT:CP_Radial_D6.3mm_P2.50mm, symbol Device:C_Polarized
- added C24: 10u, Capacitor_THT:CP_Radial_D6.3mm_P2.50mm, symbol Device:C_Polarized
- added U10, U12, U13, U14, U15, U7, U8, U9: MK4164N, Package_DIP:DIP-16_W7.62mm_Socket, symbol Memory_RAM:MK4164N
- added U4: BAT54JW-7-F, Package_TO_SOT_SMD:SOT-363_SC-70-6, symbol 2026-06-14_23-32-30:BAT54JW-7-F
- J1: MANUFACTURER_PART_NUMBER (none) -> L77HDE15SD1CH4FVGA
Connections:
- net +5V: now also C23.1, C24.1, U10.8 (VCC), U12.8 (VCC), U13.8 (VCC), U14.8 (VCC), U15.8 (VCC), U7.8 (VCC), U8.8 (VCC), U9.8 (VCC)
- net AD0: now also U10.2 (DIN)
- net AD1: now also U10.13 (A6), U12.13 (A6), U13.13 (A6), U14.13 (A6), U15.13 (A6), U7.13 (A6), U7.2 (DIN), U8.13 (A6), U9.13 (A6)
- net AD2: now also U10.10 (A5), U12.10 (A5), U13.10 (A5), U14.10 (A5), U15.10 (A5), U7.10 (A5), U8.10 (A5), U8.2 (DIN), U9.10 (A5)
- net AD3: now also U10.11 (A4), U12.11 (A4), U13.11 (A4), U14.11 (A4), U15.11 (A4), U7.11 (A4), U8.11 (A4), U9.11 (A4), U9.2 (DIN)
- net AD4: now also U10.12 (A3), U12.12 (A3), U12.2 (DIN), U13.12 (A3), U14.12 (A3), U15.12 (A3), U7.12 (A3), U8.12 (A3), U9.12 (A3)
- net AD5: now also U10.6 (A2), U12.6 (A2), U13.2 (DIN), U13.6 (A2), U14.6 (A2), U15.6 (A2), U7.6 (A2), U8.6 (A2), U9.6 (A2)
- net AD6: now also U10.7 (A1), U12.7 (A1), U13.7 (A1), U14.2 (DIN), U14.7 (A1), U15.7 (A1), U7.7 (A1), U8.7 (A1), U9.7 (A1)
- net AD7: now also U10.5 (A0), U12.5 (A0), U13.5 (A0), U14.5 (A0), U15.2 (DIN), U15.5 (A0), U7.5 (A0), U8.5 (A0), U9.5 (A0)
- net D1: no longer U3.4 (D1)
- net D2: no longer U3.7 (D2)
- net D3: no longer U3.8 (D3)
- net D4: no longer U3.13 (D4)
- net D5: no longer U3.14 (D5)
- net D6: no longer U3.17 (D6)
- net D7: no longer U3.18 (D7)
- net GND: now also U3.13 (D4), U3.14 (D5), U3.17 (D6), U3.18 (D7), U3.4 (D1), U3.7 (D2), U3.8 (D3), C23.2, C24.2, U10.16 (VSS), U10.9 (A7), U12.16 (VSS), U12.9 (A7), U13.16 (VSS), U13.9 (A7), U14.16 (VSS), U14.9 (A7), U15.16 (VSS), U15.9 (A7), U7.16 (VSS), U7.9 (A7), U8.16 (VSS), U8.9 (A7), U9.16 (VSS), U9.9 (A7)
- net R/~{W}: now also U10.3 (~{WRITE}), U12.3 (~{WRITE}), U13.3 (~{WRITE}), U14.3 (~{WRITE}), U15.3 (~{WRITE}), U7.3 (~{WRITE}), U8.3 (~{WRITE}), U9.3 (~{WRITE})
- net ~{CAS}: now also U10.15 (~{CAS}), U12.15 (~{CAS}), U13.15 (~{CAS}), U14.15 (~{CAS}), U15.15 (~{CAS}), U7.15 (~{CAS}), U8.15 (~{CAS}), U9.15 (~{CAS})
- net ~{INT}: now also U4.1 (A1)
- net ~{NMI}: now also U4.3 (A2)
- net ~{RAS}: now also U10.4 (~{RAS}), U12.4 (~{RAS}), U13.4 (~{RAS}), U14.4 (~{RAS}), U15.4 (~{RAS}), U7.4 (~{RAS}), U8.4 (~{RAS}), U9.4 (~{RAS})
- net at U5.4 (Y1): now also U4.6 (C1)
- net at U5.6 (Y0): now also U4.4 (C2)
- net VD0 renamed RD0
- net RD0: now also U10.14 (DOUT)
- net VD1 renamed RD1
- net RD1: now also U7.14 (DOUT)
- net VD2 renamed RD2
- net RD2: now also U8.14 (DOUT)
- net VD3 renamed RD3
- net RD3: now also U9.14 (DOUT)
- net VD4 renamed RD4
- net RD4: now also U12.14 (DOUT)
- net VD5 renamed RD5
- net RD5: now also U13.14 (DOUT)
- net VD6 renamed RD6
- net RD6: now also U14.14 (DOUT)
- net VD7 renamed RD7
- net RD7: now also U15.14 (DOUT)
- no-connect marks 22 -> 28
Other:
- moved on the sheet: U1A, U1B, U1C, U2B, U2D, U3

Commit message: Added bulk caps and fixed up the part numbers
Parts:
- C24: footprint Capacitor_THT:CP_Radial_D6.3mm_P2.50mm -> Capacitor_THT:CP_Radial_D5.0mm_P2.00mm; MANUFACTURER_PART_NUMBER 25YXJ220M6.3X11 -> EEA-GA1E100H
Changed lines of the file:
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@@
 			)
 		)
-		(property "Footprint" "Capacitor_THT:CP_Radial_D6.3mm_P2.50mm"
+		(property "Footprint" "Capacitor_THT:CP_Radial_D5.0mm_P2.00mm"
 			(at 171.1452 254 0)
 			(hide yes)
@@
 			)
 		)
-		(property "MANUFACTURER_PART_NUMBER" "25YXJ220M6.3X11"
+		(property "MANUFACTURER_PART_NUMBER" "EEA-GA1E100H"
 			(at 170.18 250.19 90)
 			(hide yes)
