File: Schem/LunchCrema/pBITzBusInterface.kicad_sch (KiCad schematic)
At the start: 1 part, among them J1 pBITzBus

Commit message: Nasty fix for the Lunch Crema..... the pBITz interface bus connector was mirrored!
Connections:
- net A0: now also J1.B32 (A0); no longer J1.A32 (A12)
- net A1: now also J1.B33 (A1); no longer J1.A33 (A13)
- net A2: now also J1.B34 (A2); no longer J1.A34 (A14)
- net CS0: now also J1.B21 (CS0); no longer J1.A21 (CS2)
- net CS1: now also J1.B22 (CS1); no longer J1.A22 (CS3)
- net CS2: now also J1.A21 (CS2); no longer J1.B21 (CS0)
- net CS3: now also J1.A22 (CS3); no longer J1.B22 (CS1)
- net D0: now also J1.B23 (D0); no longer J1.A23 (D8)
- net D1: now also J1.B24 (D1); no longer J1.A24 (D9)
- net D2: now also J1.B25 (D2); no longer J1.A25 (D10)
- net D3: now also J1.B26 (D3); no longer J1.A26 (D11)
- net D4: now also J1.B27 (D4); no longer J1.A27 (D12)
- net D5: now also J1.B28 (D5); no longer J1.A28 (D13)
- net D6: now also J1.B29 (D6); no longer J1.A29 (D14)
- net D7: now also J1.B30 (D7); no longer J1.A30 (D15)
- net ~{INT}: now also J1.A15 (CTRL_14); no longer J1.B15 (CTRL_4)
- net ~{NMI}: now also J1.A16 (CTRL_15); no longer J1.B16 (CTRL_5)
- net ~{RD}: now also J1.B12 (CTRL_1); no longer J1.A12 (CTRL_11)
- net ~{RESET}: now also J1.B11 (CTRL_0); no longer J1.A11 (CTRL_10)
- net ~{WAIT}: now also J1.A13 (CTRL_12); no longer J1.B13 (CTRL_2)
- net ~{WR}: now also J1.B13 (CTRL_2); no longer J1.A13 (CTRL_12)
Changed lines of the file:
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@@
+	)
+	(no_connect
+		(at 107.95 176.53)
+	)
+	(no_connect
+		(at 107.95 179.07)
 	)
 	(no_connect
@@
 	)
 	(no_connect
+		(at 107.95 199.39)
+	)
+	(no_connect
+		(at 133.35 209.55)
+	)
+	(no_connect
+		(at 133.35 158.75)
+	)
+	(no_connect
+		(at 107.95 140.97)
+	)
+	(no_connect
+		(at 133.35 219.71)
+	)
+	(no_connect
+		(at 234.95 154.94)
+	)
+	(no_connect
+		(at 133.35 151.13)
+	)
+	(no_connect
+		(at 107.95 212.09)
+	)
+	(no_connect
+		(at 107.95 194.31)
+	)
+	(no_connect
+		(at 133.35 153.67)
+	)
+	(no_connect
+		(at 107.95 191.77)
+	)
+	(no_connect
+		(at 107.95 161.29)
+	)
+	(no_connect
+		(at 133.35 217.17)
+	)
+	(no_connect
+		(at 107.95 201.93)
+	)
+	(no_connect
+		(at 107.95 229.87)
+	)
+	(no_connect
+		(at 133.35 125.73)
+	)
+	(no_connect
+		(at 107.95 125.73)
+	)
+	(no_connect
 		(at 107.95 184.15)
 	)
 	(no_connect
+		(at 107.95 156.21)
+	)
+	(no_connect
+		(at 133.35 207.01)
+	)
+	(no_connect
+		(at 133.35 229.87)
+	)
+	(no_connect
+		(at 234.95 147.32)
+	)
+	(no_connect
 		(at 107.95 186.69)
 	)
 	(no_connect
-		(at 107.95 199.39)
+		(at 107.95 189.23)
 	)
 	(no_connect
@@
 	)
 	(no_connect
-		(at 133.35 209.55)
-	)
-	(no_connect
-		(at 133.35 158.75)
-	)
-	(no_connect
-		(at 107.95 179.07)
-	)
-	(no_connect
-		(at 107.95 140.97)
-	)
-	(no_connect
-		(at 133.35 219.71)
-	)
-	(no_connect
-		(at 234.95 154.94)
-	)
-	(no_connect
-		(at 133.35 151.13)
-	)
-	(no_connect
-		(at 107.95 212.09)
-	)
-	(no_connect
-		(at 107.95 194.31)
-	)
-	(no_connect
-		(at 133.35 153.67)
-	)
-	(no_connect
-		(at 107.95 191.77)
-	)
-	(no_connect
-		(at 107.95 161.29)
-	)
-	(no_connect
-		(at 133.35 217.17)
-	)
-	(no_connect
-		(at 107.95 201.93)
-	)
-	(no_connect
-		(at 107.95 229.87)
-	)
-	(no_connect
-		(at 133.35 125.73)
-	)
-	(no_connect
-		(at 107.95 125.73)
-	)
-	(no_connect
-		(at 107.95 156.21)
-	)
-	(no_connect
-		(at 133.35 207.01)
-	)
-	(no_connect
-		(at 133.35 229.87)
-	)
-	(no_connect
-		(at 234.95 147.32)
-	)
-	(no_connect
 		(at 107.95 204.47)
 	)
@@
 	)
 	(no_connect
+		(at 133.35 214.63)
+	)
+	(no_connect
+		(at 107.95 128.27)
+	)
+	(no_connect
+		(at 267.97 154.94)
+	)
+	(no_connect
+		(at 107.95 227.33)
+	)
+	(no_connect
+		(at 107.95 153.67)
+	)
+	(no_connect
+		(at 107.95 217.17)
+	)
+	(no_connect
+		(at 107.95 219.71)
+	)
+	(no_connect
 		(at 107.95 173.99)
-	)
-	(no_connect
-		(at 133.35 214.63)
-	)
-	(no_connect
-		(at 107.95 128.27)
-	)
-	(no_connect
-		(at 107.95 189.23)
-	)
-	(no_connect
-		(at 107.95 176.53)
-	)
-	(no_connect
-		(at 267.97 154.94)
-	)
-	(no_connect
-		(at 107.95 227.33)
-	)
-	(no_connect
-		(at 107.95 153.67)
-	)
-	(no_connect
-		(at 107.95 217.17)
-	)
-	(no_connect
-		(at 107.95 219.71)
 	)
 	(no_connect
@@
 		(lib_id "pBITz:pBITzBus")
 		(at 120.65 166.37 0)
-		(mirror y)
 		(unit 1)
 		(body_style 1)
@@
 		)
 		(property "Footprint" "Connector_PCBEdge:BUS_PCIexpress_x8"
-			(at 123.698 150.876 0)
+			(at 117.602 150.876 0)
 			(hide yes)
 			(show_name no)
@@
 		)
 		(property "Datasheet" "http://www.ritrontek.com/uploadfile/2016/1026/20161026105231124.pdf#page=63"
-			(at 117.602 210.312 0)
+			(at 123.698 210.312 0)
 			(hide yes)
 			(show_name no)
@@
 		)
 		(property "Description" "pBITz backplane Connector"
-			(at 119.634 218.186 0)
-			(hide yes)
-			(show_name no)
+			(at 121.666 218.186 0)
+			(hide yes)
+			(show_name no)
