File: Schem/LunchCrema/Video.kicad_sch (KiCad schematic)
At the start: 43 parts, among them IC1 MMPQ3904, J3 DE15_Socket_HighDensity_Mount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, U10 74HC139, U2 V9958, U3 74HC273, U8 74LVC1G19, U9 BAT54JW-7-F, Y1 HC-49/U-S21477270ABJB, Y2 CPPLC5-HT7PT

Commit message: Added wait state generator to LaunchCrema
Parts:
- added C17, C18: 100n, Capacitor_SMD:C_0603_1608Metric, symbol Device:C
- added Q1: 2N7002, Package_TO_SOT_SMD:SOT-23, symbol Transistor_FET:2N7002
- added R6: 47k, Resistor_SMD:R_0603_1608Metric, symbol Device:R
- added U11: ATF22V10C-15PU, Package_DIP:DIP-24_W7.62mm_Socket, symbol Logic_Programmable:PEEL22CV10AP
- U10: value 74HC139 -> 74AHC139; MANUFACTURER_PART_NUMBER SN74HC139DR -> SN74AHC139DR
Connections:
- net +5V: now also C17.1, C18.1, U11.24 (VCC)
- net D1: now also U3.4 (D1)
- net GND: now also C17.2, C18.2, Q1.2 (S), R6.2, U11.10 (I10), U11.11 (I11), U11.12 (GND), U11.13 (I13), U11.7 (I7), U11.8 (I8), U11.9 (I9); no longer U3.4 (D1)
- net ~{CSR}: now also U11.2 (I2)
- net ~{CSW}: now also U11.3 (I3)
- net ~{RESET}: now also U11.6 (I6)
- net ~{WAIT}: now also Q1.3 (D); no longer U2.26 (~{WAIT})
- net at U2.8 (CPUCLK/VDS): now also U11.1 (I1/CLK)
- net ~{WS_EN}: now reaches U3.5 (Q1)
- net ~{WS_EN}: now also U11.5 (I5)
- new net: U11.4 (I4), U2.26 (~{WAIT})
- new net WAIT_SINK: Q1.1 (G), R6.1, U11.21 (IO21)
- no-connect marks 33 -> 40
Other:
- moved on the sheet: C10, C11, C12, C13, C14, C15, C16, C5, C8, C9

Commit message: Fixed a couple of small mistakes with the BOM
Parts:
- U10: value 74AHC139 -> 74AHCT139; MANUFACTURER_PART_NUMBER SN74AHC139DR -> SN74AHCT139DR
- U11: MANUFACTURER_PART_NUMBER (none) -> 1-2199298-8
- U3: MANUFACTURER_PART_NUMBER SN74HC273DBR -> SN74HC273DWR
- U4, U5, U6, U7: value (none) -> UPD41464C-10
Changed lines of the file:
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@@
 			)
 		)
-		(property "MANUFACTURER_PART_NUMBER" "SN74HC273DBR"
+		(property "MANUFACTURER_PART_NUMBER" "SN74HC273DWR"
 			(at 88.9 218.44 0)
 			(hide yes)
@@
 			)
 		)
-		(property "Value" ""
+		(property "Value" "UPD41464C-10"
 			(at 279.4 102.87 0)
 			(show_name no)
@@
 			)
 		)
-		(property "Value" ""
+		(property "Value" "UPD41464C-10"
 			(at 226.06 44.45 0)
 			(show_name no)
@@
 			)
 		)
-		(property "Value" ""
+		(property "Value" "UPD41464C-10"
 			(at 279.4 45.72 0)
 			(show_name no)
@@
 			)
 		)
-		(property "Value" "74AHC139"
+		(property "Value" "74AHCT139"
 			(at 88.9 281.94 0)
 			(show_name no)
@@
 			)
 		)
-		(property "MANUFACTURER_PART_NUMBER" "SN74AHC139DR"
+		(property "MANUFACTURER_PART_NUMBER" "SN74AHCT139DR"
 			(at 88.9 289.56 0)
 			(hide yes)
@@
 			)
 		)
+		(property "MANUFACTURER_PART_NUMBER" "1-2199298-8"
+			(at 96.52 129.54 0)
+			(hide yes)
+			(show_name no)
+			(do_not_autoplace no)
+			(effects
+				(font
+					(size 1.27 1.27)
+				)
+			)
+		)
 		(pin "8"
 		)
@@
 			)
 		)
-		(property "Value" "74AHC139"
+		(property "Value" "74AHCT139"
 			(at 88.9 257.81 0)
 			(show_name no)
@@
 			)
 		)
-		(property "MANUFACTURER_PART_NUMBER" "SN74AHC139DR"
+		(property "MANUFACTURER_PART_NUMBER" "SN74AHCT139DR"
 			(at 88.9 265.43 0)
 			(hide yes)
@@
 			)
 		)
-		(property "Value" ""
+		(property "Value" "UPD41464C-10"
 			(at 226.06 101.6 0)
 			(show_name no)
@@
 			)
 		)
-		(property "Value" "74AHC139"
+		(property "Value" "74AHCT139"
 			(at 58.42 421.64 90)
 			(show_name no)
@@
 			)
 		)
-		(property "MANUFACTURER_PART_NUMBER" "SN74AHC139DR"
+		(property "MANUFACTURER_PART_NUMBER" "SN74AHCT139DR"
 			(at 58.42 429.26 90)
 			(hide yes)

Commit message: updated the part #s
Parts:
- C2, C3, C4, C5: MANUFACTURER_PART_NUMBER 25YXJ220M6.3X11s -> 16YXJ220M6.3X11s
- C6, C7: MANUFACTURER_PART_NUMBER C0603C270K5RACTU -> VJ0603A270JXJPW1BC
Changed lines of the file:
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@@
 			)
 		)
-		(property "MANUFACTURER_PART_NUMBER" "C0603C270K5RACTU"
+		(property "MANUFACTURER_PART_NUMBER" "VJ0603A270JXJPW1BC"
 			(at 212.09 271.78 90)
 			(hide yes)
@@
 			)
 		)
-		(property "MANUFACTURER_PART_NUMBER" "25YXJ220M6.3X11s"
+		(property "MANUFACTURER_PART_NUMBER" "16YXJ220M6.3X11s"
 			(at 194.31 394.97 90)
 			(hide yes)
@@
 			)
 		)
-		(property "MANUFACTURER_PART_NUMBER" "25YXJ220M6.3X11s"
+		(property "MANUFACTURER_PART_NUMBER" "16YXJ220M6.3X11s"
 			(at 332.74 279.4 90)
 			(hide yes)
@@
 			)
 		)
-		(property "MANUFACTURER_PART_NUMBER" "25YXJ220M6.3X11s"
+		(property "MANUFACTURER_PART_NUMBER" "16YXJ220M6.3X11s"
 			(at 332.74 254 90)
 			(hide yes)
@@
 			)
 		)
-		(property "MANUFACTURER_PART_NUMBER" "25YXJ220M6.3X11s"
+		(property "MANUFACTURER_PART_NUMBER" "16YXJ220M6.3X11s"
 			(at 332.74 304.8 90)
 			(hide yes)
@@
 			)
 		)
-		(property "MANUFACTURER_PART_NUMBER" "C0603C270K5RACTU"
+		(property "MANUFACTURER_PART_NUMBER" "VJ0603A270JXJPW1BC"
 			(at 212.09 281.94 90)
 			(hide yes)
