File: Schem/AfternoonBlend/Sound.kicad_sch (KiCad schematic)
At the start: 56 parts, among them J4 STX-3120-3B, J5 Conn_01x03, U10 LM4880MX/NOPB, U11 SN76489AN, U12 SN76489AN, U2 TLV2372, U3 AD7801BRUZ, U6 SN76489AN, U7 SN76489AN, U8 74HC138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

Commit message: Production Information
Parts:
- C15: MANUFACTURER_PART_NUMBER CL10X106MO8NRNC -> C0603C104K5RACTU
- C17: MANUFACTURER_PART_NUMBER C0603C104K5RACTU -> CL10X106MO8NRNC
- R19, R20, R21, R22: MANUFACTURER_PART_NUMBER (none) -> RC0402FR-07100KL
- R23, R24: MANUFACTURER_PART_NUMBER RMCF0603FT10R0 -> RC0603FR-0710KL
- R30, R35: MANUFACTURER_PART_NUMBER RMCF0603FT10R0 -> CRRCR01FM47KS1
- R34, R39: MANUFACTURER_PART_NUMBER RC0603FR-0710KL -> CRRCR01FM47KS1
- U10: MANUFACTURER_PART_NUMBER (none) -> LM4880MX/NOPB
- U2: MANUFACTURER_PART_NUMBER (none) -> TLV2372IDR
- U3: MANUFACTURER_PART_NUMBER (none) -> AD7801BRUZ
- U8: MANUFACTURER_PART_NUMBER (none) -> SN74HC138DR
- U9: MANUFACTURER_PART_NUMBER (none) -> CD74HCT21M96
- Y1: MANUFACTURER_PART_NUMBER (none) -> ECS-2100A-035
Changed lines of the file:
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@@
 			)
 		)
+		(property "MANUFACTURER_PART_NUMBER" "TLV2372IDR"
+			(at 485.14 125.73 0)
+			(hide yes)
+			(show_name no)
+			(do_not_autoplace no)
+			(effects
+				(font
+					(size 1.27 1.27)
+				)
+			)
+		)
 		(pin "5"
 		)
@@
 			)
 		)
-		(property "MANUFACTURER_PART_NUMBER" ""
+		(property "MANUFACTURER_PART_NUMBER" "RC0402FR-07100KL"
 			(at 580.39 66.04 90)
 			(hide yes)
@@
 			)
 		)
+		(property "MANUFACTURER_PART_NUMBER" "AD7801BRUZ"
+			(at 292.1 64.77 0)
+			(hide yes)
+			(show_name no)
+			(do_not_autoplace no)
+			(effects
+				(font
+					(size 1.27 1.27)
+				)
+			)
+		)
 		(pin "20"
 		)
@@
 			)
 		)
+		(property "MANUFACTURER_PART_NUMBER" "CD74HCT21M96"
+			(at 71.12 231.14 0)
+			(hide yes)
+			(show_name no)
+			(do_not_autoplace no)
+			(effects
+				(font
+					(size 1.27 1.27)
+				)
+			)
+		)
 		(pin "14"
 		)
@@
 			)
 		)
-		(property "MANUFACTURER_PART_NUMBER" ""
+		(property "MANUFACTURER_PART_NUMBER" "RC0402FR-07100KL"
 			(at 450.85 175.26 90)
 			(hide yes)
@@
 			)
 		)
-		(property "MANUFACTURER_PART_NUMBER" ""
+		(property "MANUFACTURER_PART_NUMBER" "RC0402FR-07100KL"
 			(at 580.39 142.24 90)
 			(hide yes)
@@
 			)
 		)
-		(property "MANUFACTURER_PART_NUMBER" "RC0603FR-0710KL"
+		(property "MANUFACTURER_PART_NUMBER" "CRRCR01FM47KS1"
 			(at 101.6 138.43 90)
 			(hide yes)
@@
 			)
 		)
+		(property "MANUFACTURER_PART_NUMBER" "CD74HCT21M96"
+			(at 71.12 248.92 0)
+			(hide yes)
+			(show_name no)
+			(do_not_autoplace no)
+			(effects
+				(font
+					(size 1.27 1.27)
+				)
+			)
+		)
 		(pin "14"
 		)
@@
 			)
 		)
+		(property "MANUFACTURER_PART_NUMBER" "TLV2372IDR"
+			(at 482.6 177.8 0)
+			(hide yes)
+			(show_name no)
+			(do_not_autoplace no)
+			(effects
+				(font
+					(size 1.27 1.27)
+				)
+			)
+		)
 		(pin "5"
 		)
@@
 			)
 		)
+		(property "MANUFACTURER_PART_NUMBER" "CD74HCT21M96"
+			(at 40.64 252.73 0)
+			(hide yes)
+			(show_name no)
+			(do_not_autoplace no)
+			(effects
+				(font
+					(size 1.27 1.27)
+				)
+			)
+		)
 		(pin "14"
 		)
@@
 			)
 		)
-		(property "MANUFACTURER_PART_NUMBER" "RMCF0603FT10R0"
+		(property "MANUFACTURER_PART_NUMBER" "CRRCR01FM47KS1"
 			(at 388.62 78.74 0)
 			(hide yes)
@@
 			)
 		)
+		(property "MANUFACTURER_PART_NUMBER" "TLV2372IDR"
+			(at 483.87 55.88 0)
+			(hide yes)
+			(show_name no)
+			(do_not_autoplace no)
+			(effects
+				(font
+					(size 1.27 1.27)
+				)
+			)
+		)
 		(pin "5"
 		)
@@
 			)
 		)
+		(property "MANUFACTURER_PART_NUMBER" "ECS-2100A-035"
+			(at 133.35 308.61 0)
+			(hide yes)
+			(show_name no)
+			(do_not_autoplace no)
+			(effects
+				(font
+					(size 1.27 1.27)
+				)
+			)
+		)
 		(pin "8"
 		)
@@
 			)
 		)
-		(property "MANUFACTURER_PART_NUMBER" "CL10X106MO8NRNC"
+		(property "MANUFACTURER_PART_NUMBER" "C0603C104K5RACTU"
 			(at 546.1 139.7 90)
 			(hide yes)
@@
 			)
 		)
-		(property "MANUFACTURER_PART_NUMBER" "RMCF0603FT10R0"
+		(property "MANUFACTURER_PART_NUMBER" "CRRCR01FM47KS1"
 			(at 388.62 67.31 0)
 			(hide yes)
@@
 			)
 		)
-		(property "MANUFACTURER_PART_NUMBER" ""
+		(property "MANUFACTURER_PART_NUMBER" "RC0402FR-07100KL"
 			(at 462.28 167.64 90)
 			(hide yes)
@@
 			)
 		)
-		(property "MANUFACTURER_PART_NUMBER" "C0603C104K5RACTU"
+		(property "MANUFACTURER_PART_NUMBER" "CL10X106MO8NRNC"
 			(at 100.33 308.61 0)
 			(hide yes)
@@
 			)
 		)
+		(property "MANUFACTURER_PART_NUMBER" "LM4880MX/NOPB"
+			(at 541.02 128.27 90)
+			(hide yes)
+			(show_name no)
+			(do_not_autoplace no)
+			(effects
+				(font
+					(size 1.27 1.27)
+				)
+			)
+		)
 		(pin "8"
 		)
@@
 			)
 		)
-		(property "MANUFACTURER_PART_NUMBER" "RC0603FR-0710KL"
+		(property "MANUFACTURER_PART_NUMBER" "CRRCR01FM47KS1"
 			(at 217.17 134.62 90)
 			(hide yes)
@@
 			)
 		)
-		(property "MANUFACTURER_PART_NUMBER" "RMCF0603FT10R0"
+		(property "MANUFACTURER_PART_NUMBER" "RC0603FR-0710KL"
 			(at 495.3 137.16 0)
 			(hide yes)
@@
 			)
 		)
+		(property "MANUFACTURER_PART_NUMBER" "SN74HC138DR"
+			(at 137.16 251.46 0)
+			(hide yes)
+			(show_name no)
+			(do_not_autoplace no)
+			(effects
+				(font
+					(size 1.27 1.27)
+				)
+			)
+		)
 		(pin "2"
 		)
@@
 			)
 		)
-		(property "MANUFACTURER_PART_NUMBER" "RMCF0603FT10R0"
+		(property "MANUFACTURER_PART_NUMBER" "RC0603FR-0710KL"
 			(at 495.3 67.31 0)
 			(hide yes)
