File: Schem/AfternoonBlend/AfternoonBlend.kicad_pcb (KiCad board)
At the start: 4 copper layers, 160 x 70 mm, 72 parts, among them J4 STX-3120-3B, J5 Conn_01x03, Q1 2N7002, SW1 SW_Coded_SH-7070, U1 74HC688, U10 LM4880MX/NOPB, U11 SN76489AN, U12 SN76489AN, U14 74HC20, U2 TLV2372, U3 AD7801BRUZ, U4 74HCT541, U5 74AHCT74, U6 SN76489AN, U7 SN76489AN, U8 74AHCT138, U9 74AHCT00, Y1 ECS-2100A-035

Commit message: Fab on 6 layers for panelization
Routing:
- added copper zone on In3.Cu, net GND
- added copper zone on In4.Cu, net GND
Other:
- copper layers 4 -> 6
Changed lines of the file:
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@@
 		(4 "In1.Cu" power)
 		(6 "In2.Cu" power)
+		(8 "In3.Cu" power)
+		(10 "In4.Cu" power)
 		(2 "B.Cu" signal)
 		(9 "F.Adhes" user "F.Adhesive")
@@
 			)
 			(layer "dielectric 2"
-				(type "core")
-				(thickness 1.24)
+				(type "prepreg")
+				(thickness 0.535)
 				(material "FR4")
 				(epsilon_r 4.5)
@@
 				(loss_tangent 0.02)
 			)
+			(layer "In3.Cu"
+				(type "copper")
+				(thickness 0.035)
+			)
+			(layer "dielectric 4"
+				(type "prepreg")
+				(color "#808080FF")
+				(thickness 0.535)
+				(material "FR4")
+				(epsilon_r 4.5)
+				(loss_tangent 0.02)
+			)
+			(layer "In4.Cu"
+				(type "copper")
+				(thickness 0.035)
+			)
+			(layer "dielectric 5"
+				(type "prepreg")
+				(thickness 0.1)
+				(material "FR4")
+				(epsilon_r 4.5)
+				(loss_tangent 0.02)
+			)
 			(layer "B.Cu"
 				(type "copper")
@@
 		(capping no)
 		(filling no)
+		(zone_defaults)
 		(aux_axis_origin 53.78444 155.911135)
 		(grid_origin 82.35 51.22)
@@
 			)
 		)
+	)
+	(zone
+		(net "GND")
+		(layers "In3.Cu" "In4.Cu")
+		(hatch edge 0.5)
+		(priority 2)
+		(connect_pads
+			(clearance 0.5)
+		)
+		(min_thickness 0.25)
+		(fill yes
+			(thermal_gap 0.5)
+			(thermal_bridge_width 0.5)
+			(island_removal_mode 0)
+		)
+		(polygon
+			(pts
+				(xy 63.7794 58.2582) (xy 223.7794 58.2582) (xy 223.7794 128.2582) (xy 64.1614 128.2582)
+			)
+		)

Commit message: updated the part #s
Parts:
- removed REF**: OSHW-Logo2_7.3x6mm_SilkScreen, Symbol:OSHW-Logo2_7.3x6mm_SilkScreen
Routing:
- removed copper zone on In3.Cu, net GND
- removed copper zone on In4.Cu, net GND
Other:
- copper layers 6 -> 4
